File: ESP12S-measure-v2/esp8266-bme280-deepsleep.sch (EAGLE design)
At the start: 21 parts, among them U1 74HC4051D,653

Commit message: The board now goes to deep sleep and not in soft ap, if the ssid cannot be found. This is crucial, so that it does not drain the battery.
Parts:
- CLEAR, FLASH, RESET: value B3U-1000P -> SWCH-SMD-1; device B3U-1000P:B3U-1000P -> SMD-SWITCH-1:SWCH-SMD-1
Changed lines of the file:
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@@
 <part name="SUPPLY8" library="supply2" library_urn="urn:adsk.eagle:library:372" deviceset="VCC" device=""/>
 <part name="GND10" library="supply1" library_urn="urn:adsk.eagle:library:371" deviceset="GND" device=""/>
-<part name="FLASH" library="B3U-1000P" deviceset="B3U-1000P" device=""/>
-<part name="CLEAR" library="B3U-1000P" deviceset="B3U-1000P" device=""/>
-<part name="RESET" library="B3U-1000P" deviceset="B3U-1000P" device=""/>
+<part name="FLASH" library="SMD-SWITCH-1" deviceset="SWCH-SMD-1" device=""/>
+<part name="CLEAR" library="SMD-SWITCH-1" deviceset="SWCH-SMD-1" device=""/>
+<part name="RESET" library="SMD-SWITCH-1" deviceset="SWCH-SMD-1" device=""/>
 <part name="AN1" library="con-lstb" library_urn="urn:adsk.eagle:library:162" deviceset="MA03-1" device="" package3d_urn="urn:adsk.eagle:package:8339/1"/>
 <part name="AN2" library="con-lstb" library_urn="urn:adsk.eagle:library:162" deviceset="MA03-1" device="" package3d_urn="urn:adsk.eagle:package:8339/1"/>
